Commit message: Eliminate xacro warning

File: fake_joint_driver/robot/arm3.urdf.xacro (robot description, xacro)
@@ -1,5 +1,5 @@
 <?xml version="1.0"?>
 <robot xmlns:xacro="http://ros.org/wiki/xacro" name="arm3">
-  <property name="M_PI" value="3.1415926535897931" />
+  <xacro:property name="M_PI" value="3.1415926535897931" />
   <link name="arm3"/>
   <joint name="JOINT1" type="revolute">
